File: hardware/schematic/kicad/power.kicad_sch (KiCad schematic)
At the start: 119 parts, among them J101 12-15V DC, Q101 IPD25N06S4L-30, Q102 IPD25N06S4L-30, Q103 IPD33CN10N, Q104 MMBTA06, U101 LT3757EMSE, U102 LT3757EMSE, U103 LT3757EMSE, U104 TPS7A4701 +16V, U105 TPS7A3301 -16V, U106 TPS7A4701 +5V, U107 LT3042 +3V3A, U108 TPS62130, U109 TPS62130, U110 TLV75518 +1V8

Commit message: Add footprints and starting PCB so Altium import resolves every part
Altium's ECO reported "Footprint Not Found" for every part (and the
resulting "Unknown Pin" / class-member errors) because only KiCad
footprint names were included. Now:

- aio.kicad_pcb: every part placed with its footprint, all pads on their
  nets (unrouted), generated by pcb.py
- aio.pretty/: the 45 footprints the design uses, bundled with the project
- footprint fixes: five names that did not exist in the KiCad library
  replaced (coupled inductors -> two SRR1260 per converter, SRP5030T,
  RK097 dual pot, NCJ6FI-H, DPDT gain switch); parts without an explicit
  footprint now keep the symbol's default; phantom switch moved from a
  momentary push-button to a latching slide switch
- check.py also verifies every PCB pad's net against design.py
- README: Altium import steps (full project, then Make PCB Library)

U203 (XU316) still has no footprint: its pin numbers are placeholders
until the official XMOS library part replaces it.
Parts:
- added L109, L110: 2.2u, Inductor_SMD:L_Bourns_SRP5030T, symbol Device:L
- L101: value 2x22u 1:1 -> 22u 4A; footprint Inductor_SMD:L_Coupled_Coilcraft_MSD1278 -> Inductor_SMD:L_Bourns_SRR1260; symbol Device:L_Coupled -> Device:L; MPN MSD1278-223MLB -> SRR1260-220M
- L102, L104: value 1u -> 22u 4A; footprint Inductor_SMD:L_1210_3225Metric -> Inductor_SMD:L_Bourns_SRR1260; MPN (none) -> SRR1260-220M
- L103: value 2x22u 1:1 -> 1u; footprint Inductor_SMD:L_Coupled_Coilcraft_MSD1278 -> Inductor_SMD:L_1210_3225Metric; symbol Device:L_Coupled -> Device:L; MPN MSD1278-223MLB -> (none)
- L105: value 22u -> 22u 4A; MPN (none) -> SRR1260-220M
- L106: value 10u -> 1u
- L107: value 2.2u -> 22u; footprint Inductor_SMD:L_Bourns_SRP4020TA -> Inductor_SMD:L_Bourns_SRR1260
- L108: value 2.2u -> 10u; footprint Inductor_SMD:L_Bourns_SRP4020TA -> Inductor_SMD:L_1210_3225Metric
- U104, U105, U106: footprint (none) -> Package_DFN_QFN:Texas_RGW0020A_VQFN-20-1EP_5x5mm_P0.65mm_EP3.15x3.15mm_ThermalVias
- U107: footprint (none) -> Package_SO:MSOP-10-1EP_3x3mm_P0.5mm_EP1.68x1.88mm
- U108, U109: footprint (none) -> Package_DFN_QFN:VQFN-16-1EP_3x3mm_P0.5mm_EP1.68x1.68mm_ThermalVias
Connections:
- net +0V9: now also L110.2; no longer L108.2
- net +18V4: now also L103.2; no longer L102.2
- net +18V4_SW: now also L103.1; no longer L102.1
- net +3V3D: now also L109.2; no longer L107.2
- net +50V: now also L108.2; no longer L106.2
- net +50V_SW: now also L108.1; no longer L106.1
- net -18V4: now also L106.2; no longer L104.2
- net -18V4_SW: now also L105.1, L106.1; no longer L103.3, L104.1
- net GND: now also L102.1; no longer L101.3
- net SW2: now also L104.2; no longer L103.2
- net SW3: now also L107.2; no longer L105.2
- net SW_0V9: now also L110.1; no longer L108.1
- net SW_3V3: now also L109.1; no longer L107.1
- net VIN: now also L104.1, L107.1; no longer L103.1, L105.1
- net X1: now also L102.2; no longer L101.4
- net X2: now also L105.2; no longer L103.4
Other:
- moved on the sheet: C108, C109, C110, C111, C112, C113, C114, C115, C116, C117, C118, C119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
