File: hardware/schematic/kicad/usb.kicad_sch (KiCad schematic)
At the start: 52 parts, among them J201 USB-C, J202 DEBUG (verify), Q201 AO3407A, U201 TPD4E05U06, U202 STUSB4500, U203 XU316-1024-QF60B, U204 W25Q32JVSS, U205 74LVC1G3157, X201 24.000MHz, X202 24.576MHz, X203 22.5792MHz

Commit message: Add footprints and starting PCB so Altium import resolves every part
Altium's ECO reported "Footprint Not Found" for every part (and the
resulting "Unknown Pin" / class-member errors) because only KiCad
footprint names were included. Now:

- aio.kicad_pcb: every part placed with its footprint, all pads on their
  nets (unrouted), generated by pcb.py
- aio.pretty/: the 45 footprints the design uses, bundled with the project
- footprint fixes: five names that did not exist in the KiCad library
  replaced (coupled inductors -> two SRR1260 per converter, SRP5030T,
  RK097 dual pot, NCJ6FI-H, DPDT gain switch); parts without an explicit
  footprint now keep the symbol's default; phantom switch moved from a
  momentary push-button to a latching slide switch
- check.py also verifies every PCB pad's net against design.py
- README: Altium import steps (full project, then Make PCB Library)

U203 (XU316) still has no footprint: its pin numbers are placeholders
until the official XMOS library part replaces it.
Parts:
- U201: footprint (none) -> Package_SON:USON-10_2.5x1.0mm_P0.5mm
- U202: footprint (none) -> Package_DFN_QFN:QFN-24-1EP_4x4mm_P0.5mm_EP2.7x2.7mm
- U203: footprint Package_DFN_QFN:QFN-60-1EP_7x7mm_P0.4mm -> (none)
- U204: footprint (none) -> Package_SO:SOIC-8_5.23x5.23mm_P1.27mm
- X201, X202, X203: footprint (none) -> Oscillator:Oscillator_SMD_Abracon_ASE-4Pin_3.2x2.5mm
Changed lines of the file:
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@@
       )
     )
-    (property "Footprint" ""
+    (property "Footprint" "Package_SON:USON-10_2.5x1.0mm_P0.5mm"
       (at 144.78 38.1 0)
       (effects
@@
       )
     )
-    (property "Footprint" ""
+    (property "Footprint" "Package_DFN_QFN:QFN-24-1EP_4x4mm_P0.5mm_EP2.7x2.7mm"
       (at 193.04 63.5 0)
       (effects
@@
       )
     )
-    (property "Footprint" "Package_DFN_QFN:QFN-60-1EP_7x7mm_P0.4mm"
+    (property "Footprint" ""
       (at 50.8 152.4 0)
       (effects
@@
       )
     )
-    (property "Footprint" ""
+    (property "Footprint" "Oscillator:Oscillator_SMD_Abracon_ASE-4Pin_3.2x2.5mm"
       (at 510.54 121.92 0)
       (effects
@@
       )
     )
-    (property "Footprint" ""
+    (property "Footprint" "Package_SO:SOIC-8_5.23x5.23mm_P1.27mm"
       (at 43.18 231.14 0)
       (effects
@@
       )
     )
-    (property "Footprint" ""
+    (property "Footprint" "Oscillator:Oscillator_SMD_Abracon_ASE-4Pin_3.2x2.5mm"
       (at 137.16 226.06 0)
       (effects
@@
       )
     )
-    (property "Footprint" ""
+    (property "Footprint" "Oscillator:Oscillator_SMD_Abracon_ASE-4Pin_3.2x2.5mm"
       (at 175.26 226.06 0)
       (effects
