File: hardware/schematic/kicad/dac.kicad_sch (KiCad schematic)
At the start: 50 parts, among them U301 PCM1794A, U302 OPA1612, U303 OPA1612, U304 OPA1612

Commit message: Add footprints and starting PCB so Altium import resolves every part
Altium's ECO reported "Footprint Not Found" for every part (and the
resulting "Unknown Pin" / class-member errors) because only KiCad
footprint names were included. Now:

- aio.kicad_pcb: every part placed with its footprint, all pads on their
  nets (unrouted), generated by pcb.py
- aio.pretty/: the 45 footprints the design uses, bundled with the project
- footprint fixes: five names that did not exist in the KiCad library
  replaced (coupled inductors -> two SRR1260 per converter, SRP5030T,
  RK097 dual pot, NCJ6FI-H, DPDT gain switch); parts without an explicit
  footprint now keep the symbol's default; phantom switch moved from a
  momentary push-button to a latching slide switch
- check.py also verifies every PCB pad's net against design.py
- README: Altium import steps (full project, then Make PCB Library)

U203 (XU316) still has no footprint: its pin numbers are placeholders
until the official XMOS library part replaces it.
Parts:
- RV301: footprint Potentiometer_THT:Potentiometer_Alps_RK27_Dual_Horizontal -> Potentiometer_THT:Potentiometer_Alps_RK097_Dual_Horizontal; MPN ALPS RK27112A 10KAX2 -> ALPS RK097 dual 10k log (A)
- U301: footprint (none) -> Package_SO:SSOP-28_5.3x10.2mm_P0.65mm
Changed lines of the file:
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@@
       )
     )
-    (property "Footprint" ""
+    (property "Footprint" "Package_SO:SSOP-28_5.3x10.2mm_P0.65mm"
       (at 53.34 60.96 0)
       (effects
@@
       )
     )
-    (property "Footprint" "Potentiometer_THT:Potentiometer_Alps_RK27_Dual_Horizontal"
+    (property "Footprint" "Potentiometer_THT:Potentiometer_Alps_RK097_Dual_Horizontal"
       (at 530.86 157.48 0)
       (effects
@@
       )
     )
-    (property "MPN" "ALPS RK27112A 10KAX2"
+    (property "MPN" "ALPS RK097 dual 10k log (A)"
       (at 530.86 157.48 0)
       (effects

Commit message: Split schematic into 14 A3 sheets, fix board outline, cluster placement
- Schematic: the five large A1/A0 sheets become 14 A3 sheets, one per
  function. Designators are unchanged (sections share one numbering
  sequence); the BOM is identical.
- PCB staging board: the outline was computed from board edges before any
  existed, so it came out far too small. It now encloses all parts. Parts
  are packed into one labelled cluster per sheet instead of one long strip.
- README: Altium steps for the "Missing child-sheet" errors (drop the top
  sheet, use global net scope) and layout guidance: don't autoroute the
  staging board.
Parts:
- removed C311, C312, C315, C316: 2.2n C0G, Capacitor_SMD:C_0603_1608Metric, symbol Device:C
- removed C313, C314, C317, C318, C319, C320: 100n, Capacitor_SMD:C_0603_1608Metric, symbol Device:C
- removed C321, C322, C324, C325: 1.5n C0G, Capacitor_SMD:C_0603_1608Metric, symbol Device:C
- removed C323, C326: 4.7u film, Capacitor_THT:C_Rect_L18.0mm_W8.0mm_P15.00mm_FKS3_FKP3, symbol Device:C
- removed R308, R309, R310, R311: 750R 0.1%, Resistor_SMD:R_0603_1608Metric, symbol Device:R
- removed R312, R314, R316, R318: 2.00k 0.1%, Resistor_SMD:R_0603_1608Metric, symbol Device:R
- removed R313, R315, R317, R319: 1.00k 0.1%, Resistor_SMD:R_0603_1608Metric, symbol Device:R
- removed RV301: 10k log dual, Potentiometer_THT:Potentiometer_Alps_RK097_Dual_Horizontal, symbol Device:R_Potentiometer_Dual
- removed U302, U303, U304: OPA1612, Package_SO:SOIC-8_3.9x4.9mm_P1.27mm, symbol Amplifier_Operational:OPA1612AxD
Other:
- title: DAC, I/V, volume -> DAC (PCM1794A)
- moved on the sheet: C302, C303, C306, C308, C309, R301, R302, R303, R304, R305, R306, R307
