File: hardware/schematic/kicad/aio.kicad_pcb (KiCad board)
At the start: 2 copper layers, 10.1 x 153.7 mm, 356 parts, among them J101 12-15V DC, J201 USB-C, J202 DEBUG (verify), J401 6.35mm, J402 3.5mm, J501 NCJ6FI-H, K401 G6K-2F-Y 3VDC, Q101 IPD25N06S4L-30, Q102 IPD25N06S4L-30, Q103 IPD33CN10N, Q104 MMBTA06, Q201 AO3407A, Q401 2N7002, Q402 BC847, Q403 BC847, SW401 GAIN H/L, SW501 +48V, U101 LT3757EMSE, U102 LT3757EMSE, U103 LT3757EMSE, U104 TPS7A4701 +16V, U105 TPS7A3301 -16V, U106 TPS7A4701 +5V, U107 LT3042 +3V3A, U108 TPS62130, U109 TPS62130, U110 TLV75518 +1V8, U201 TPD4E05U06, U202 STUSB4500, U204 W25Q32JVSS, U205 74LVC1G3157, U301 PCM1794A, U302 OPA1612, U303 OPA1612, U304 OPA1612, U401 OPA1612, U402 LME49600, U403 LME49600, U404 LME49600, U405 LME49600, U406 LM393, U501 THAT1512S08, U502 OPA1612, U503 CS5361, X201 24.000MHz, X202 24.576MHz, X203 22.5792MHz

Commit message: Split schematic into 14 A3 sheets, fix board outline, cluster placement
- Schematic: the five large A1/A0 sheets become 14 A3 sheets, one per
  function. Designators are unchanged (sections share one numbering
  sequence); the BOM is identical.
- PCB staging board: the outline was computed from board edges before any
  existed, so it came out far too small. It now encloses all parts. Parts
  are packed into one labelled cluster per sheet instead of one long strip.
- README: Altium steps for the "Missing child-sheet" errors (drop the top
  sheet, use global net scope) and layout guidance: don't autoroute the
  staging board.
Parts:
- moved Q402 307.2 mm to (297.3, 100.5)
- moved R431 307.2 mm to (291.8, 99.3)
- moved C140 250.2 mm to (288.2, 4.75)
- moved U105 250.2 mm to (266.5, 7.15)
- moved C137 250.2 mm to (246.2, 5.62)
- moved C138 250.2 mm to (256.0, 8.43)
- moved C139 250.2 mm to (278.1, 4.75)
- moved R123 250.2 mm to (273.1, 4.75)
- moved R124 250.2 mm to (283.1, 4.75)
- moved J402 236.4 mm to (274.6, 115.2)
- moved Q403 236.4 mm to (236.5, 111.3)
- moved R432 236.4 mm to (231.1, 110.2)
- moved J401 236.4 mm to (247.8, 111.5)
- moved K401 223.2 mm to (234.2, 91.3)
- moved C420 223.2 mm to (286.8, 86.8)
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Other:
- board size 10.1 x 153.7 mm -> 311.5 x 253.2 mm
- board text added: "+50V boost and +48V phantom supply"
- board text added: "-18V4 Cuk converter"
- board text added: "ADC driver and ADC (CS5361)"
- board text added: "Audio master clocks, I2S, LEDs"
- board text added: "DAC (PCM1794A)"
- board text added: "DAC I/V stage, output filter, volume"
- board text added: "Digital supplies: +3V3D, +0V9, +1V8"
- board text added: "Headphone amplifier"
- board text added: "Linear regulators: +-16V, +5VA, +3V3A"
- board text added: "Microphone input, phantom feed, preamp"
- board text added: "Output relay, protection, headphone jacks"
- board text added: "Power input and +18V4 SEPIC converter"
- board text added: "USB-C connector and PD sink"
- board text added: "XMOS XU316, boot flash, debug"

Commit message: Place components by function on a 200 x 130 mm board
place.py replaces the staging layout with a real first-pass placement:
- floorplan: switchers back-left, LDOs as a buffer strip, digital/USB/XMOS/
  clocks/DAC at the back right, mic + ADC front-left, headphone amp and
  protection front-right
- panel parts (DC jack, USB-C, XLR, jacks, pots, switches, LEDs) on the
  edges, rotated so the mating face points out
- ICs spread in their region, each passive next to the pin it connects to;
  decoupling caps anchor to the IC they are drawn with (median 3.7 mm from
  the supply pin, 90% within 7.7 mm)
- corners kept clear for mounting holes, no courtyard overlaps, everything
  inside the outline; region outlines on Cmts.User
Parts:
- moved C147 240.1 mm to (59.5, 77.2)
- moved R125 234.5 mm to (59.3, 74.0), turned to 90 degrees
- moved U107 232.0 mm to (54.7, 73.0)
- moved C140 218.4 mm to (76.3, 57.8), turned to 90 degrees
- moved R124 213.3 mm to (75.4, 53.0)
- moved C139 211.5 mm to (72.4, 53.9), turned to 90 degrees
- moved L108 211.1 mm to (12.9, 77.0)
- moved R123 209.7 mm to (69.4, 54.3)
- moved R119 207.0 mm to (4.28, 62.8), turned to 90 degrees
- moved C131 204.5 mm to (10.0, 66.8), turned to 90 degrees
- moved C137 203.5 mm to (49.4, 57.7), turned to 90 degrees
- moved U105 201.3 mm to (72.0, 59.0)
- moved C138 199.2 mm to (63.0, 57.7), turned to 90 degrees
- moved C130 194.9 mm to (13.7, 67.8), turned to 90 degrees
- moved C146 192.4 mm to (84.3, 57.2), turned to 90 degrees
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Other:
- board size 311.5 x 253.2 mm -> 200 x 130 mm
